File: Browse/t1.kicad_pcb (KiCad board)
At the start: 4 copper layers, 63 x 35.6 mm, 47 parts, among them J1 Barrel_Jack_Switch, J2 USB_B, J3 P1, J4 2x2M, J5 ICSP1, J6 P2, U1 ATmega8U2-AU, Y1 16MHz

Commit message: Deploying to main from @ INTI-CMNB/kibot_variants_arduprog@d882be12f9a46b3037afef0ba314bb9c105903a5 🚀
Routing:
- net Net-(F1-Pad2): track 10.3 -> 9.49 mm
