File: Browse/t1.kicad_sch (KiCad schematic)
At the start: 47 parts, among them J1 Barrel_Jack_Switch, J2 USB_B, J3 P1, J4 2x2M, J5 ICSP1, J6 P2, U1 ATmega8U2-AU, Y1 16MHz

Commit message: Deploying to main from @ INTI-CMNB/kibot_variants_arduprog@d882be12f9a46b3037afef0ba314bb9c105903a5 🚀
Other:
- moved on the sheet: FID1, FID2, FID3, FID4, H1, H2, H3, H4
