File: Browse/t1.kicad_sch (KiCad schematic)
At the start: 47 parts, among them J1 Barrel_Jack_Switch, J2 USB_B, J3 P1, J4 2x2M, J5 ICSP1, J6 P2, U1 ATmega8U2-AU, Y1 16MHz

Commit message: Deploying to main from @ INTI-CMNB/kibot_variants_arduprog@0931c6eb52cb798f53ae0dbc289b20b281a80a9d 🚀
Parts:
- J3: symbol Connector:Conn_01x05_Male -> Connector:Conn_01x05_Pin
- J6: symbol Connector:Conn_01x06_Male -> Connector:Conn_01x06_Pin

Commit message: Deploying to main from @ INTI-CMNB/kibot_variants_arduprog@68529856bb4947410f10c31e01fa79e07a02a501 🚀
Parts:
- C1: MFN Vishay Beyschlag/Draloric/BC Components -> (none); MFP MAL215371479E3 -> (none); MNF (none) -> Vishay Beyschlag/Draloric/BC Components; MPN (none) -> MAL215371479E3
- D2, D3: MFN OSRAM Opto Semiconductors Inc. -> (none); MFP LG R971-KN-1 -> (none); MNF (none) -> OSRAM Opto Semiconductors Inc.; MPN (none) -> LG R971-KN-1
- FB1: MFN Murata -> (none); MFP BLM21PG221SN1D -> (none); MNF (none) -> Murata; MPN (none) -> BLM21PG221SN1D
- J1: MFN Würth Elektronik -> (none); MFP 694106106102 -> (none); MNF (none) -> Würth Elektronik; MPN (none) -> 694106106102
- J2: MFN TE Connectivity AMP Connectors -> (none); MFP 292304-1 -> (none); MNF (none) -> TE Connectivity AMP Connectors; MPN (none) -> 292304-1
- J4: MFN Harwin Inc. -> (none); MFP M20-9980246-ND -> (none); MNF (none) -> Harwin Inc.; MPN (none) -> M20-9980246-ND
- J5: MFN Harwin Inc. -> (none); MFP M20-9980346 -> (none); MNF (none) -> Harwin Inc.; MPN (none) -> M20-9980346
- VR1, VR2: MFN Bourns Inc. -> (none); MFP CG0603MLC-05E -> (none); MNF (none) -> Bourns Inc.; MPN (none) -> CG0603MLC-05E
- Y1: MFN Abracon LLC -> (none); MFP ABM3-16.000MHZ-B2-T -> (none); MNF (none) -> Abracon LLC; MPN (none) -> ABM3-16.000MHZ-B2-T
Changed lines of the file:
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@@
       (effects (font (size 1.27 1.27)) (hide yes))
     )
-    (property "MFN" "Bourns Inc." (at 100.33 119.38 0)
-      (effects (font (size 1.27 1.27)) (hide yes))
-    )
-    (property "MFP" "CG0603MLC-05E" (at 100.33 119.38 0)
+    (property "MNF" "Bourns Inc." (at 100.33 119.38 0)
+      (effects (font (size 1.27 1.27)) (hide yes))
+    )
+    (property "MPN" "CG0603MLC-05E" (at 100.33 119.38 0)
       (effects (font (size 1.27 1.27)) (hide yes))
     )
@@
       (effects (font (size 1.27 1.27)) (hide yes))
     )
-    (property "MFN" "Abracon LLC" (at 120.65 80.01 90)
-      (effects (font (size 1.27 1.27)) (hide yes))
-    )
-    (property "MFP" "ABM3-16.000MHZ-B2-T" (at 120.65 80.01 90)
+    (property "MNF" "Abracon LLC" (at 120.65 80.01 90)
+      (effects (font (size 1.27 1.27)) (hide yes))
+    )
+    (property "MPN" "ABM3-16.000MHZ-B2-T" (at 120.65 80.01 90)
       (effects (font (size 1.27 1.27)) (hide yes))
     )
@@
       (effects (font (size 1.27 1.27)) (hide yes))
     )
-    (property "Datasheet" "~" (at 76.2 109.22 0)
+    (property "Datasheet" " ~" (at 76.2 109.22 0)
       (effects (font (size 1.27 1.27)) (hide yes))
     )
@@
       (effects (font (size 1.27 1.27)) (hide yes))
     )
-    (property "MFN" "TE Connectivity AMP Connectors" (at 72.39 107.95 0)
-      (effects (font (size 1.27 1.27)) (hide yes))
-    )
-    (property "MFP" "292304-1" (at 72.39 107.95 0)
+    (property "MNF" "TE Connectivity AMP Connectors" (at 72.39 107.95 0)
+      (effects (font (size 1.27 1.27)) (hide yes))
+    )
+    (property "MPN" "292304-1" (at 72.39 107.95 0)
       (effects (font (size 1.27 1.27)) (hide yes))
     )
@@
       (effects (font (size 1.27 1.27)) (hide yes))
     )
-    (property "MFN" "Bourns Inc." (at 91.44 119.38 0)
-      (effects (font (size 1.27 1.27)) (hide yes))
-    )
-    (property "MFP" "CG0603MLC-05E" (at 91.44 119.38 0)
+    (property "MNF" "Bourns Inc." (at 91.44 119.38 0)
+      (effects (font (size 1.27 1.27)) (hide yes))
+    )
+    (property "MPN" "CG0603MLC-05E" (at 91.44 119.38 0)
       (effects (font (size 1.27 1.27)) (hide yes))
     )
@@
       (effects (font (size 1.27 1.27)) (hide yes))
     )
-    (property "MFN" "Murata" (at 96.52 130.81 0)
-      (effects (font (size 1.27 1.27)) (hide yes))
-    )
-    (property "MFP" "BLM21PG221SN1D" (at 96.52 130.81 0)
+    (property "MNF" "Murata" (at 96.52 130.81 0)
+      (effects (font (size 1.27 1.27)) (hide yes))
+    )
+    (property "MPN" "BLM21PG221SN1D" (at 96.52 130.81 0)
       (effects (font (size 1.27 1.27)) (hide yes))
     )
@@
       (effects (font (size 1.27 1.27)) (hide yes))
     )
-    (property "MFN" "OSRAM Opto Semiconductors Inc." (at 248.92 115.57 90)
-      (effects (font (size 1.27 1.27)) (hide yes))
-    )
-    (property "MFP" "LG R971-KN-1" (at 248.92 115.57 90)
+    (property "MNF" "OSRAM Opto Semiconductors Inc." (at 248.92 115.57 90)
+      (effects (font (size 1.27 1.27)) (hide yes))
+    )
+    (property "MPN" "LG R971-KN-1" (at 248.92 115.57 90)
       (effects (font (size 1.27 1.27)) (hide yes))
     )
@@
       (effects (font (size 1.27 1.27)) (hide yes))
     )
-    (property "MFN" "Würth Elektronik" (at 54.61 50.8 0)
-      (effects (font (size 1.27 1.27)) (hide yes))
-    )
-    (property "MFP" "694106106102" (at 54.61 50.8 0)
+    (property "MNF" "Würth Elektronik" (at 54.61 50.8 0)
+      (effects (font (size 1.27 1.27)) (hide yes))
+    )
+    (property "MPN" "694106106102" (at 54.61 50.8 0)
       (effects (font (size 1.27 1.27)) (hide yes))
     )
@@
       (effects (font (size 1.27 1.27)) (hide yes))
     )
-    (property "MFN" "Harwin Inc." (at 213.36 74.93 0)
-      (effects (font (size 1.27 1.27)) (hide yes))
-    )
-    (property "MFP" "M20-9980346" (at 213.36 74.93 0)
+    (property "MNF" "Harwin Inc." (at 213.36 74.93 0)
+      (effects (font (size 1.27 1.27)) (hide yes))
+    )
+    (property "MPN" "M20-9980346" (at 213.36 74.93 0)
       (effects (font (size 1.27 1.27)) (hide yes))
     )
@@
       (effects (font (size 1.27 1.27)) (hide yes))
     )
-    (property "MFN" "Harwin Inc." (at 208.28 86.36 0)
-      (effects (font (size 1.27 1.27)) (hide yes))
-    )
-    (property "MFP" "M20-9980246-ND" (at 208.28 86.36 0)
+    (property "MNF" "Harwin Inc." (at 208.28 86.36 0)
+      (effects (font (size 1.27 1.27)) (hide yes))
+    )
+    (property "MPN" "M20-9980246-ND" (at 208.28 86.36 0)
       (effects (font (size 1.27 1.27)) (hide yes))
     )
@@
       (effects (font (size 1.27 1.27)) (hide yes))
     )
-    (property "MFN" "OSRAM Opto Semiconductors Inc." (at 236.22 115.57 90)
-      (effects (font (size 1.27 1.27)) (hide yes))
-    )
-    (property "MFP" "LG R971-KN-1" (at 236.22 115.57 90)
+    (property "MNF" "OSRAM Opto Semiconductors Inc." (at 236.22 115.57 90)
+      (effects (font (size 1.27 1.27)) (hide yes))
+    )
+    (property "MPN" "LG R971-KN-1" (at 236.22 115.57 90)
       (effects (font (size 1.27 1.27)) (hide yes))
     )
@@
       (effects (font (size 1.27 1.27)) (hide yes))
     )
-    (property "MFN" "Vishay Beyschlag/Draloric/BC Components" (at 82.55 53.34 0)
-      (effects (font (size 1.27 1.27)) (hide yes))
-    )
-    (property "MFP" "MAL215371479E3" (at 82.55 53.34 0)
+    (property "MNF" "Vishay Beyschlag/Draloric/BC Components" (at 82.55 53.34 0)
+      (effects (font (size 1.27 1.27)) (hide yes))
+    )
+    (property "MPN" "MAL215371479E3" (at 82.55 53.34 0)
       (effects (font (size 1.27 1.27)) (hide yes))
     )
@@
       (effects (font (size 1.27 1.27)) (hide yes))
     )
+    (property "Sim.Enable" "0" (at 71.755 166.37 0)
+      (effects (font (size 1.27 1.27)) (hide yes))
+    )
