File: Browse/t1.kicad_sch (KiCad schematic)
At the start: 47 parts, among them J1 Barrel_Jack_Switch, J2 USB_B, J3 P1, J4 2x2M, J5 ICSP1, J6 P2, U1 ATmega8U2-AU, Y1 16MHz

Commit message: Deploying to main from @ INTI-CMNB/kibot_variants_arduprog@92cc0c668f1c59fe53a319740111dce91ed73298 🚀
Parts:
- C1: MFN (none) -> Vishay Beyschlag/Draloric/BC Components; MFP (none) -> MAL215371479E3; MNF Vishay Beyschlag/Draloric/BC Components -> (none); MPN MAL215371479E3 -> (none)
- D2, D3: MFN (none) -> OSRAM Opto Semiconductors Inc.; MFP (none) -> LG R971-KN-1; MNF OSRAM Opto Semiconductors Inc. -> (none); MPN LG R971-KN-1 -> (none)
- FB1: MFN (none) -> Murata; MFP (none) -> BLM21PG221SN1D; MNF Murata -> (none); MPN BLM21PG221SN1D -> (none)
- J1: MFN (none) -> Würth Elektronik; MFP (none) -> 694106106102; MNF Würth Elektronik -> (none); MPN 694106106102 -> (none)
- J2: MFN (none) -> TE Connectivity AMP Connectors; MFP (none) -> 292304-1; MNF TE Connectivity AMP Connectors -> (none); MPN 292304-1 -> (none)
- J4: MFN (none) -> Harwin Inc.; MFP (none) -> M20-9980246-ND; MNF Harwin Inc. -> (none); MPN M20-9980246-ND -> (none)
- J5: MFN (none) -> Harwin Inc.; MFP (none) -> M20-9980346; MNF Harwin Inc. -> (none); MPN M20-9980346 -> (none)
- VR1, VR2: MFN (none) -> Bourns Inc.; MFP (none) -> CG0603MLC-05E; MNF Bourns Inc. -> (none); MPN CG0603MLC-05E -> (none)
- Y1: MFN (none) -> Abracon LLC; MFP (none) -> ABM3-16.000MHZ-B2-T; MNF Abracon LLC -> (none); MPN ABM3-16.000MHZ-B2-T -> (none)
Other:
- company: Instituto Nacional de Tecnología Industrial -> Arduino
- moved on the sheet: FID1, FID2, FID3, FID4, H1, H2, H3, H4
